Commit message: Better linearization implementation

File: gazebo_worlds/urdf/herbie.xacro (robot description, xacro)
@@ -8,10 +8,10 @@
         <inertial>
             <mass value="0.7"/>
-            <origin rpy="0 0 0" xyz="0.05 0 0.074"/>
+            <origin rpy="0 0 0" xyz="-0.15 0 0.074"/>
             <xacro:box_inertia mass="0.7" x="0.22" y="0.147" z="0.10"/>
         </inertial>
         <!-- body -->
         <collision name="collision_chassis">
-            <origin rpy="0 0 0" xyz="0.05 0 0.074"/>
+            <origin rpy="0 0 0" xyz="-0.15 0 0.074"/>
             <geometry>
                 <box size="0.22 0.147 0.10"/>
@@ -19,5 +19,5 @@
         </collision>
         <visual>
-            <origin rpy="0 0 0" xyz="0.05 0 0.074"/>
+            <origin rpy="0 0 0" xyz="-0.15 0 0.074"/>
             <geometry>
                 <box size="0.22 0.147 0.10"/>
@@ -94,5 +94,5 @@
     </link>
     <joint name="joint_right_wheel" type="continuous">
-        <origin rpy="-1.5708 0 0" xyz="0.0 -0.054 0.03125"/>
+        <origin rpy="-1.5708 0 0" xyz="-0.2 -0.054 0.03125"/>
         <child link="link_right_wheel"/>
         <parent link="link_chassis"/>
@@ -102,5 +102,5 @@
     </joint>
     <joint name="joint_left_wheel" type="continuous">
-        <origin rpy="-1.5708 0 0" xyz="0.0 0.054 0.03125"/>
+        <origin rpy="-1.5708 0 0" xyz="-0.2 0.054 0.03125"/>
         <child link="link_left_wheel"/>
         <parent link="link_chassis"/>
@@ -110,5 +110,5 @@
     </joint>
     <joint name="joint_caster_wheel" type="continuous">
-        <origin rpy="-1.5708 0 0" xyz="0.15 0 0.012"/>
+        <origin rpy="-1.5708 0 0" xyz="-0.05 0 0.012"/>
         <child link="link_caster_wheel"/>
         <parent link="link_chassis"/>
